File: KiCad/V1/GameboyCartridgeV1.1/power.kicad_sch (KiCad schematic)
At the start: 22 parts, among them Q1 CJ2302, U4 CartBus, U5 MCP1825T-3302E/DC, U6 TXB0102DCU, U7 TXB0108PW, U8 TXB0108PW, U9 TXB0108PW

Commit message: Change folder structure
- Fix Library paths
- Add Libraries
- Add Gerbers, BOM, Position file compatible with JLPCB
Parts:
- added FID1, FID2, FID3: Fiducial, Fiducial:Fiducial_1mm_Mask2mm, symbol Mechanical:Fiducial
- D2: renamed from D1; LCSC (none) -> C669022
- D3: renamed from D2; LCSC (none) -> C669022
- Q1: LCSC (none) -> C8548
- U3: renamed from U4; now left out of the parts list
- U4: renamed from U5; LCSC (none) -> C632684
- U5: renamed from U6; LCSC (none) -> C60709
- U6: renamed from U7; LCSC (none) -> C53406
- U7: renamed from U8; LCSC (none) -> C53406
- U8: renamed from U9; LCSC (none) -> C53406
- renumbered C13 to C15, C14 to C16, C15 to C17, C16 to C18, C17 to C19, C18 to C20, C19 to C21, C20 to C22, C21 to C23, C22 to C24, R10 to R7, R11 to R8, R12 to R9
